File: boards/RocketBlaster_v3.0/RocketBlaster_v3.0.kicad_pcb (KiCad board)
At the start: 2 copper layers, 62.2 x 26.7 mm, 28 parts, among them J0 Conn_02x03_Odd_Even, J1 B2B-XH-A_LF__SN_, J2 B2B-XH-A_LF__SN_, J3 B2B-XH-A_LF__SN_, J4 B2B-XH-A_LF__SN_, J5 B2B-XH-A_LF__SN_, Q1 IRLML6344TRPBF, U1 ATMEGA328PB-AU, U2 LM7805MPX_NOPB, U3 DFR0299

Commit message: Corrections to schematic and PCB parameters for OSH Park
Parts:
- R3: value 220R -> 100R
- R4, R5: value 1kOhm -> 1k
- U3: value DFR0299 -> DFPlayer Mini
Other:
- rule pad_to_mask_clearance: 0.051 -> 0.0508
- rule solder_mask_min_width: 0.25 -> 0.1016
- rule trace_min: 0.2 -> 0.1524
- rule via_min_drill: 0.3 -> 0.254
- rule via_min_size: 0.4 -> 0.508
