File: boards/RocketBlaster_v3.0/RocketBlaster_v3.0.sch (KiCad schematic (older format))
At the start: 24 parts, among them J0 Conn_02x03_Odd_Even, J1 B2B-XH-A_LF__SN_, J2 B2B-XH-A_LF__SN_, J3 B2B-XH-A_LF__SN_, J4 B2B-XH-A_LF__SN_, J5 B2B-XH-A_LF__SN_, Q1 IRLML6344TRPBF, U1 ATMEGA328PB-AU, U2 LM7805MPX_NOPB, U3 DFR0299

Commit message: Corrections to schematic and PCB parameters for OSH Park
Parts:
- U3: value DFR0299 -> DFPlayer Mini; footprint MODULE_DFR0299 -> DFR0299:MODULE_DFR0299
Connections:
- no-connect marks 0 -> 25
Changed lines of the file:
@@
 P 9350 3500
 F 0 "U3" H 9350 4367 50  0000 C CNN
-F 1 "DFR0299" H 9350 4276 50  0000 C CNN
-F 2 "MODULE_DFR0299" H 9350 3500 50  0001 L BNN
+F 1 "DFPlayer Mini" H 9350 4276 50  0000 C CNN
+F 2 "DFR0299:MODULE_DFR0299" H 9350 3500 50  0001 L BNN
 F 3 "Dfplayer - a Mini Mp3 Player" H 9350 3500 50  0001 L BNN
 F 4 "DFR0299" H 9350 3500 50  0001 L BNN "Field4"
@@
 Text Notes 7400 7500 0    50   ~ 0
 RocketBlaster v3.0
+NoConn ~ 9950 3100
+NoConn ~ 9950 3200
+NoConn ~ 9950 3700
+NoConn ~ 9950 3800
+NoConn ~ 8750 3300
+NoConn ~ 8750 3400
+NoConn ~ 8750 3600
+NoConn ~ 8750 3700
+NoConn ~ 5450 1900
+NoConn ~ 5650 2400
+NoConn ~ 5650 2500
+NoConn ~ 5650 2600
+NoConn ~ 5650 3100
+NoConn ~ 5650 3200
+NoConn ~ 5650 3300
+NoConn ~ 4850 3700
+NoConn ~ 4850 3400
+NoConn ~ 4850 3300
+NoConn ~ 4850 3200
+NoConn ~ 4850 3100
+NoConn ~ 4850 3000
+NoConn ~ 4850 2900
+NoConn ~ 4850 2800
+NoConn ~ 4850 2700
+NoConn ~ 4850 2300
 $EndSCHEMATC

Commit message: Update KiCAD files, add enclosure folder, and add README info
Parts:
- D1: symbol dk_Diodes-Rectifiers-Single:S1G -> RocketBlaster_v3.0-rescue:S1G-dk_Diodes-Rectifiers-Single
- J1, J2, J3, J4, J5: symbol dk_Rectangular-Connectors-Headers-Male-Pins:B2B-XH-A_LF__SN_ -> RocketBlaster_v3.0-rescue:B2B-XH-A_LF__SN_-dk_Rectangular-Connectors-Headers-Male-Pins
- L1, L2, L3: symbol dk_LED-Indication-Discrete:151033RS03000 -> RocketBlaster_v3.0-rescue:151033RS03000-dk_LED-Indication-Discrete
- Q1: symbol dk_Transistors-FETs-MOSFETs-Single:IRLML6344TRPBF -> RocketBlaster_v3.0-rescue:IRLML6344TRPBF-dk_Transistors-FETs-MOSFETs-Single
- U1: symbol dk_Embedded-Microcontrollers:ATMEGA328PB-AU -> RocketBlaster_v3.0-rescue:ATMEGA328PB-AU-dk_Embedded-Microcontrollers
- U2: symbol LM7805MPX_NOPB:LM7805MPX_NOPB -> RocketBlaster_v3.0-rescue:LM7805MPX_NOPB-LM7805MPX_NOPB
- U3: symbol DFR0299:DFR0299 -> RocketBlaster_v3.0-rescue:DFR0299-DFR0299
Changed lines of the file:
@@
 $EndDescr
 $Comp
-L dk_Embedded-Microcontrollers:ATMEGA328PB-AU U1
+L RocketBlaster_v3.0-rescue:ATMEGA328PB-AU-dk_Embedded-Microcontrollers U1
 U 1 1 5E2652CB
 P 5350 2500
@@
 $EndComp
 $Comp
-L dk_Rectangular-Connectors-Headers-Male-Pins:B2B-XH-A_LF__SN_ J1
+L RocketBlaster_v3.0-rescue:B2B-XH-A_LF__SN_-dk_Rectangular-Connectors-Headers-Male-Pins J1
 U 1 1 5E268083
 P 1550 1700
@@
 $EndComp
 $Comp
-L dk_LED-Indication-Discrete:151033RS03000 L1
+L RocketBlaster_v3.0-rescue:151033RS03000-dk_LED-Indication-Discrete L1
 U 1 1 5E269ADF
 P 2150 5950
@@
 $EndComp
 $Comp
-L dk_LED-Indication-Discrete:151033RS03000 L2
+L RocketBlaster_v3.0-rescue:151033RS03000-dk_LED-Indication-Discrete L2
 U 1 1 5E26B28B
 P 2150 5300
@@
 $EndComp
 $Comp
-L dk_LED-Indication-Discrete:151033RS03000 L3
+L RocketBlaster_v3.0-rescue:151033RS03000-dk_LED-Indication-Discrete L3
 U 1 1 5E26CE74
 P 2150 4650
@@
 $EndComp
 $Comp
-L LM7805MPX_NOPB:LM7805MPX_NOPB U2
+L RocketBlaster_v3.0-rescue:LM7805MPX_NOPB-LM7805MPX_NOPB U2
 U 1 1 5E26DC82
 P 7300 1650
@@
 $EndComp
 $Comp
-L dk_Transistors-FETs-MOSFETs-Single:IRLML6344TRPBF Q1
+L RocketBlaster_v3.0-rescue:IRLML6344TRPBF-dk_Transistors-FETs-MOSFETs-Single Q1
 U 1 1 5E273C51
 P 7400 5150
@@
 $EndComp
 $Comp
-L DFR0299:DFR0299 U3
+L RocketBlaster_v3.0-rescue:DFR0299-DFR0299 U3
 U 1 1 5E279048
 P 9350 3500
@@
 $EndComp
 $Comp
-L dk_Diodes-Rectifiers-Single:S1G D1
+L RocketBlaster_v3.0-rescue:S1G-dk_Diodes-Rectifiers-Single D1
 U 1 1 5E28151C
 P 6950 4550
@@
 VREG
 $Comp
-L dk_Rectangular-Connectors-Headers-Male-Pins:B2B-XH-A_LF__SN_ J2
+L RocketBlaster_v3.0-rescue:B2B-XH-A_LF__SN_-dk_Rectangular-Connectors-Headers-Male-Pins J2
 U 1 1 5E29C425
 P 1550 2100
@@
 SW_ARM
 $Comp
-L dk_Rectangular-Connectors-Headers-Male-Pins:B2B-XH-A_LF__SN_ J3
+L RocketBlaster_v3.0-rescue:B2B-XH-A_LF__SN_-dk_Rectangular-Connectors-Headers-Male-Pins J3
 U 1 1 5E2B930D
 P 1550 2500
@@
 SW_GO
 $Comp
-L dk_Rectangular-Connectors-Headers-Male-Pins:B2B-XH-A_LF__SN_ J4
+L RocketBlaster_v3.0-rescue:B2B-XH-A_LF__SN_-dk_Rectangular-Connectors-Headers-Male-Pins J4
 U 1 1 5E2BA1C6
 P 4050 4750
@@
 TRG
 $Comp
-L dk_Rectangular-Connectors-Headers-Male-Pins:B2B-XH-A_LF__SN_ J5
+L RocketBlaster_v3.0-rescue:B2B-XH-A_LF__SN_-dk_Rectangular-Connectors-Headers-Male-Pins J5
 U 1 1 5E3007CC
 P 7300 4500
